File: src/Engine-Controller/USB.sch (KiCad schematic (older format))
At the start: 0 parts

Commit message: Annotated Schematic
Parts:
- added J2: USB, BEL_SS-52300-001, symbol Engine-Controller:USB
Connections:
- new net 5V: J2.1 (VCC)
- new net Earth: J2.4 (GND)
Changed lines of the file:
@@
 $Descr A4 11693 8268
 encoding utf-8
-Sheet 1 5
-Title ""
-Date ""
-Rev ""
-Comp ""
-Comment1 ""
+Sheet 3 5
+Title "Liquids Engine Microcontroller USB"
+Date "2021-06-29"
+Rev "1.0"
+Comp "Sun Devil Rocketry "
+Comment1 "Author: Colton Acosta"
 Comment2 ""
 Comment3 ""
 Comment4 ""
 $EndDescr
+$Comp
+L Engine-Controller:USB J2
+U 1 1 60FB1D93
+P 5300 4200
+F 0 "J2" H 5193 4767 50  0000 C CNN
+F 1 "USB" H 5193 4676 50  0000 C CNN
+F 2 "BEL_SS-52300-001" H 4950 3600 50  0001 L BNN
+F 3 "" H 5300 4200 50  0001 L BNN
+	1    5300 4200
+	-1   0    0    -1
+$EndComp
+$Comp
+L power:Earth #PWR0110
+U 1 1 60FB3329
+P 5950 4600
+F 0 "#PWR0110" H 5950 4350 50  0001 C CNN
+F 1 "Earth" H 5950 4450 50  0001 C CNN
+F 2 "" H 5950 4600 50  0001 C CNN
+F 3 "~" H 5950 4600 50  0001 C CNN
+	1    5950 4600
+	1    0    0    -1
+$EndComp
+Wire Wire Line
+	5700 4200 5950 4200
+Wire Wire Line
+	5950 4200 5950 4600
+Text GLabel 6200 3900 2    50   Input ~ 0
+5V
+Wire Wire Line
+	5700 3900 6200 3900
 $EndSCHEMATC
